File: mcu_main/display.kicad_sch (KiCad schematic)
At the start: 0 parts

Commit message: Added connections for the display SPI
Parts:
- added J9: Conn_01x14_Socket, Connector_Molex:Molex_KK-254_AE-6410-14A_1x14_P2.54mm_Vertical, symbol Connector:Conn_01x14_Socket
Connections:
- new net +5V: J9.1 (Pin_1)
- new net Display_CLK: J9.7 (Pin_7)
- new net Display_CS: J9.3 (Pin_3)
- new net Display_DC/RS: J9.5 (Pin_5)
- new net Display_LED: J9.8 (Pin_8)
- new net Display_MISO: J9.9 (Pin_9)
- new net Display_MOSI: J9.6 (Pin_6)
- new net Display_RST: J9.4 (Pin_4)
- new net Display_T_CLK: J9.10 (Pin_10)
- new net Display_T_CS: J9.11 (Pin_11)
- new net Display_T_DIN: J9.12 (Pin_12)
- new net Display_T_DO: J9.13 (Pin_13)
- new net Display_T_IRQ: J9.14 (Pin_14)
- new net GND: J9.2 (Pin_2)

Commit message: started pcb layout
Parts:
- J9: footprint Connector_Molex:Molex_KK-254_AE-6410-14A_1x14_P2.54mm_Vertical -> Connector_PinHeader_2.54mm:PinHeader_1x14_P2.54mm_Vertical
Changed lines of the file:
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@@
 			)
 		)
-		(property "Footprint" "Connector_Molex:Molex_KK-254_AE-6410-14A_1x14_P2.54mm_Vertical"
+		(property "Footprint" "Connector_PinHeader_2.54mm:PinHeader_1x14_P2.54mm_Vertical"
 			(at 142.24 95.25 0)
 			(effects
