File: mcu_main/pas_sensor.kicad_sch (KiCad schematic)
At the start: 1 part, among them J8 Screw_Terminal_01x06

Commit message: added most things to the pcb, review required
Connections:
- net speed_sig_1: now also J8.3 (Pin_3); no longer J8.4 (Pin_4)
- net speed_sig_2: now also J8.4 (Pin_4); no longer J8.3 (Pin_3)
Changed lines of the file:
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@@
+	(wire
+		(pts
+			(xy 129.54 96.52) (xy 111.76 96.52)
+		)
+		(stroke
+			(width 0)
+			(type default)
+		)
+	)
 	(wire
 		(pts
@@
 	(wire
 		(pts
-			(xy 129.54 96.52) (xy 111.76 96.52)
+			(xy 111.76 96.52) (xy 111.76 95.25)
 		)
 		(stroke
@@
 		(pts
 			(xy 128.27 101.6) (xy 129.54 101.6)
-		)
-		(stroke
-			(width 0)
-			(type default)
-		)
-	)
-	(wire
-		(pts
-			(xy 111.76 96.52) (xy 111.76 95.25)
 		)
 		(stroke
@@
 	(hierarchical_label "speed_sig_1"
 		(shape input)
-		(at 128.27 104.14 180)
+		(at 128.27 101.6 180)
 		(effects
 			(font
@@
 	(hierarchical_label "speed_sig_2"
 		(shape input)
-		(at 128.27 101.6 180)
+		(at 128.27 104.14 180)
 		(effects
 			(font
